File: kicad/LEDs.sch (KiCad schematic (older format))
At the start: 59 parts, among them U10 WS2812B, U11 WS2812B, U12 WS2812B, U13 WS2812B, U14 WS2812B, U15 WS2812B, U16 WS2812B, U17 WS2812B, U18 WS2812B, U19 WS2812B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

Commit message: Updated hardware design and removed test idf-code
Parts:
- renumbered C11 to C10, C12 to C11, C13 to C12, C14 to C13, C15 to C14, C16 to C15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
