File: kicad/sensors.sch (KiCad schematic (older format))
At the start: 16 parts, among them J10 OLED, J9 Gesture, U34 APDS-9960, U35 MMA8452Q

Commit message: Updated hardware design and removed test idf-code
Parts:
- removed C42: 4.7uF, Capacitors_SMD:C_0805_HandSoldering, symbol C
- removed C43, C44: 0.1uF, Capacitors_SMD:C_0603_HandSoldering, symbol C
- removed R16: 4k7, Resistors_SMD:R_0603_HandSoldering, symbol R
- removed U35: MMA8452Q, QFN16:QFN-16, symbol MMA8452Q
- added J11: MMA8542Q Accelerometer, Pin_Headers:Pin_Header_Straight_1x08_Pitch2.54mm, symbol Conn_01x08
- added R14: 4k7, Resistors_SMD:R_0603_HandSoldering, symbol R
- renumbered C39 to C38, C40 to C39, C41 to C40, R11 to R10, R12 to R11, R13 to R12, R14 to R13, U34 to U33
Connections:
- net +3V3: now also J11.2 (Pin_2), R14.1
- net GND: now also J11.3 (Pin_3)
- net INT1: now also J11.7 (Pin_7)
- net INT2: now also J11.8 (Pin_8); no longer R15.2
- net SCL1: now also J11.4 (Pin_4), R14.2
- net SDA1: now also R15.2, J11.5 (Pin_5)
- no-connect marks 0 -> 2
